File: Radio/Radio.kicad_sch (KiCad schematic)
At the start: 2 parts, among them J1 CON-SMA-EDGE-S, U1 RFM95W-868S2

Commit message: Add files via upload
Connections:
- net Interrupt GPIO Pin: now reaches U1.14 (DIO0)
- net GPIO PIN : now reaches U1.6 (RESET)
- net 3.3 V renamed +3.3V
- no-connect marks 0 -> 5
