File: PowerReg/PowerReg.kicad_sch (KiCad schematic)
At the start: 6 parts, among them U2 TPS62172DSG

Commit message: Add files via upload
Parts:
- removed C1: C, symbol Device:C
- removed C2: 22uF, symbol Device:C
- removed L1: 2.2uH, symbol Device:L
- removed R1: 100k, symbol Device:R
- removed U2: TPS62172DSG, Package_SON:WSON-8-1EP_2x2mm_P0.5mm_EP0.9x1.6mm_ThermalVias, symbol Regulator_Switching:TPS62172DSG
- added C3: 10uF, symbol Device:C
- added C4: 22uF, symbol Device:C
- added L2: 2.2uH, symbol Device:L
- added R2: 100k, symbol Device:R
- added U1: TPS62162DSG, Package_SON:WSON-8-1EP_2x2mm_P0.5mm_EP0.9x1.6mm_ThermalVias, symbol Regulator_Switching:TPS62162DSG
Connections:
- net GND: now also BT1.2 (-), C3.2, C4.1, C4.2, L2.2, R2.1, U1.1 (PGND), U1.4 (AGND), U1.5 (FB), U1.6 (VOS), U1.9 (PAD)
- net Vin: now also C3.1, U1.2 (VIN), U1.3 (EN)
- new net: L2.1, U1.7 (SW)
- new net PG: R2.2, U1.8 (PG)
Other:
- moved on the sheet: BT1

Commit message: Add files via upload
Parts:
- removed BT1: 3.7V, symbol Device:Battery_Cell
Connections:
- net GND: no longer C4.1, L2.2, R2.1, U1.5 (FB), U1.6 (VOS)
- new net +3.3V: C4.1, L2.2, R2.1, U1.5 (FB), U1.6 (VOS)
Other:
- moved on the sheet: C4
Changed lines of the file:
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@@
 	(paper "A4")
-	(junction
-		(at 175.26 62.23)
-		(diameter 0)
-		(color 0 0 0 0)
-	)
 	(junction
 		(at 143.51 59.69)
@@
 		(color 0 0 0 0)
 	)
-	(wire
-		(pts
-			(xy 175.26 62.23) (xy 175.26 71.12)
-		)
-		(stroke
-			(width 0)
-			(type default)
-		)
+	(junction
+		(at 162.56 62.23)
+		(diameter 0)
+		(color 0 0 0 0)
+	)
+	(junction
+		(at 177.8 62.23)
+		(diameter 0)
+		(color 0 0 0 0)
 	)
 	(wire
@@
 	(wire
 		(pts
+			(xy 162.56 62.23) (xy 177.8 62.23)
+		)
+		(stroke
+			(width 0)
+			(type default)
+		)
+	)
+	(wire
+		(pts
 			(xy 123.19 74.93) (xy 123.19 77.47)
 		)
@@
 	(wire
 		(pts
-			(xy 143.51 62.23) (xy 175.26 62.23)
-		)
-		(stroke
-			(width 0)
-			(type default)
-		)
-	)
-	(wire
-		(pts
-			(xy 86.36 57.15) (xy 86.36 63.5)
+			(xy 143.51 62.23) (xy 162.56 62.23)
 		)
 		(stroke
@@
 	(wire
 		(pts
+			(xy 177.8 69.85) (xy 177.8 71.12)
+		)
+		(stroke
+			(width 0)
+			(type default)
+		)
+	)
+	(wire
+		(pts
 			(xy 96.52 77.47) (xy 120.65 77.47)
 		)
@@
 	(wire
 		(pts
+			(xy 177.8 53.34) (xy 177.8 62.23)
+		)
+		(stroke
+			(width 0)
+			(type default)
+		)
+	)
+	(wire
+		(pts
 			(xy 143.51 57.15) (xy 148.59 57.15)
 		)
@@
 	(wire
 		(pts
-			(xy 175.26 60.96) (xy 175.26 62.23)
-		)
-		(stroke
-			(width 0)
-			(type default)
-		)
-	)
-	(wire
-		(pts
 			(xy 106.68 57.15) (xy 113.03 57.15)
 		)
@@
 	(wire
 		(pts
-			(xy 175.26 53.34) (xy 187.96 53.34)
-		)
-		(stroke
-			(width 0)
-			(type default)
-		)
-	)
-	(wire
-		(pts
-			(xy 86.36 71.12) (xy 86.36 73.66)
+			(xy 85.09 58.42) (xy 88.9 58.42)
+		)
+		(stroke
+			(width 0)
+			(type default)
+		)
+	)
+	(wire
+		(pts
+			(xy 162.56 54.61) (xy 162.56 62.23)
+		)
+		(stroke
+			(width 0)
+			(type default)
+		)
+	)
+	(wire
+		(pts
+			(xy 177.8 53.34) (xy 187.96 53.34)
 		)
 		(stroke
@@
 	)
 	(label "Vin"
-		(at 86.36 57.15 0)
+		(at 96.52 59.69 0)
 		(fields_autoplaced yes)
 		(effects
@@
 		)
 	)
-	(label "Vin"
-		(at 96.52 59.69 0)
+	(label "PG"
+		(at 111.76 67.31 0)
 		(fields_autoplaced yes)
 		(effects
@@
 		)
 	)
-	(label "PG"
-		(at 111.76 67.31 0)
+	(label "Vin"
+		(at 106.68 59.69 0)
 		(fields_autoplaced yes)
 		(effects
@@
 		)
 	)
-	(label "Vin"
-		(at 106.68 59.69 0)
+	(global_label "Vin"
+		(shape input)
+		(at 85.09 58.42 180)
 		(fields_autoplaced yes)
 		(effects
@@
 				(size 1.27 1.27)
 			)
-			(justify left bottom)
+			(justify right)
+		)
+		(property "Intersheetrefs" "${INTERSHEET_REFS}"
+			(at 79.2624 58.42 0)
+			(effects
+				(font
+					(size 1.27 1.27)
+				)
+				(justify right)
+				(hide yes)
+			)
 		)
 	)
@@
 	)
 	(symbol
-		(lib_id "power:GND")
-		(at 86.36 73.66 0)
+		(lib_id "power:+3.3V")
+		(at 162.56 54.61 0)
 		(unit 1)
 		(exclude_from_sim no)
@@
 		(dnp no)
 		(fields_autoplaced yes)
-		(property "Reference" "#PWR04"
-			(at 86.36 80.01 0)
-			(effects
-				(font
-					(size 1.27 1.27)
-				)
-				(hide yes)
-			)
-		)
-		(property "Value" "GND"
-			(at 86.36 78.74 0)
+		(property "Reference" "#PWR01"
+			(at 162.56 58.42 0)
+			(effects
+				(font
+					(size 1.27 1.27)
+				)
+				(hide yes)
+			)
+		)
+		(property "Value" "+3.3V"
+			(at 162.56 49.53 0)
 			(effects
 				(font
@@
 		)
 		(property "Footprint" ""
-			(at 86.36 73.66 0)
+			(at 162.56 54.61 0)
 			(effects
 				(font
@@
 		)
 		(property "Datasheet" ""
-			(at 86.36 73.66 0)
-			(effects
-				(font
-					(size 1.27 1.27)
-				)
-				(hide yes)
-			)
-		)
-		(property "Description" "Power symbol creates a global label with name \"GND\" , ground"
-			(at 86.36 73.66 0)
+			(at 162.56 54.61 0)
+			(effects
+				(font
+					(size 1.27 1.27)
+				)
+				(hide yes)
+			)
+		)
+		(property "Description" "Power symbol creates a global label with name \"+3.3V\""
+			(at 162.56 54.61 0)
 			(effects
 				(font
@@
 		)
 		(instances
-			(project "PowerReg"
+			(project ""
 				(path "/69b89bc5-ef32-4b14-b574-fcede0ff2705"
-					(reference "#PWR04")
+					(reference "#PWR01")
 					(unit 1)
 				)
@@
 	)
 	(symbol
-		(lib_id "Device:Battery_Cell")
-		(at 86.36 68.58 0)
-		(unit 1)
-		(exclude_from_sim no)
-		(in_bom yes)
-		(on_board yes)
-		(dnp no)
-		(fields_autoplaced yes)
-		(property "Reference" "BT1"
-			(at 90.17 65.4684 0)
-			(effects
-				(font
-					(size 1.27 1.27)
-				)
-				(justify left)
-			)
-		)
-		(property "Value" "3.7V"
-			(at 90.17 68.0084 0)
-			(effects
-				(font
-					(size 1.27 1.27)
-				)
-				(justify left)
-			)
-		)
-		(property "Footprint" ""
-			(at 86.36 67.056 90)
-			(effects
-				(font
-					(size 1.27 1.27)
-				)
-				(hide yes)
-			)
-		)
-		(property "Datasheet" "~"
-			(at 86.36 67.056 90)
-			(effects
-				(font
-					(size 1.27 1.27)
-				)
-				(hide yes)
-			)
-		)
-		(property "Description" "Single-cell battery"
-			(at 86.36 68.58 0)
-			(effects
-				(font
-					(size 1.27 1.27)
-				)
-				(hide yes)
-			)
-		)
-		(pin "1"
-		)
-		(pin "2"
-		)
-		(instances
-			(project ""
-				(path "/69b89bc5-ef32-4b14-b574-fcede0ff2705"
-					(reference "BT1")
-					(unit 1)
-				)
-			)
-		)
-	)
-	(symbol
 		(lib_id "Device:L")
 		(at 139.7 57.15 90)
@@
 	(symbol
 		(lib_id "power:GND")
-		(at 175.26 71.12 0)
+		(at 177.8 71.12 0)
 		(unit 1)
 		(exclude_from_sim no)
@@
 		(fields_autoplaced yes)
 		(property "Reference" "#PWR05"
-			(at 175.26 77.47 0)
+			(at 177.8 77.47 0)
 			(effects
 				(font
@@
 		)
 		(property "Value" "GND"
-			(at 175.26 76.2 0)
+			(at 177.8 76.2 0)
 			(effects
 				(font
@@
 		)
 		(property "Footprint" ""
-			(at 175.26 71.12 0)
+			(at 177.8 71.12 0)
 			(effects
 				(font
@@
 		)
 		(property "Datasheet" ""
-			(at 175.26 71.12 0)
+			(at 177.8 71.12 0)
 			(effects
 				(font
@@
 		)
 		(property "Description" "Power symbol creates a global label with name \"GND\" , ground"
-			(at 175.26 71.12 0)
+			(at 177.8 71.12 0)
 			(effects
 				(font
@@
 	(symbol
 		(lib_id "Device:C")
-		(at 175.26 57.15 0)
+		(at 177.8 66.04 0)
 		(unit 1)
 		(exclude_from_sim no)
@@
 		(fields_autoplaced yes)
 		(property "Reference" "C4"
-			(at 179.07 55.8799 0)
+			(at 181.61 64.7699 0)
 			(effects
 				(font
@@
 		)
 		(property "Value" "22uF"
-			(at 179.07 58.4199 0)
+			(at 181.61 67.3099 0)
 			(effects
 				(font
@@
 		)
 		(property "Footprint" ""
-			(at 176.2252 60.96 0)
+			(at 178.7652 69.85 0)
 			(effects
 				(font
@@
 		)
 		(property "Datasheet" "~"
-			(at 175.26 57.15 0)
+			(at 177.8 66.04 0)
 			(effects
 				(font
@@
 		)
 		(property "Description" "Unpolarized capacitor"
-			(at 175.26 57.15 0)
-			(effects
-				(font
+			(at 177.8 66.04 0)
+			(effects
+				(font

Commit message: Add files via upload
Parts:
- C3, C4: footprint (none) -> Capacitor_SMD:C_0201_0603Metric
- L2: footprint (none) -> Inductor_SMD:L_1008_2520Metric
- R2: footprint (none) -> Resistor_SMD:R_0402_1005Metric
Connections:
- net +3.3V: no longer U1.5 (FB)
- net GND: now also U1.5 (FB)
- net Vin renamed +BATT
Other:
- moved on the sheet: C4, R2
