File: KiCad/LNA_IN.kicad_sch (KiCad schematic)
At the start: 6 parts

Commit message: very rough sketch layout
Parts:
- AE1: renamed from AE2; footprint (none) -> RF_Antenna:Molex_47948-0001_2.4Ghz
- C15: renamed from C11; footprint (none) -> Capacitor_SMD:C_0402_1005Metric
- C16: renamed from C12; footprint (none) -> Capacitor_SMD:C_0402_1005Metric
- C17: renamed from C13; footprint (none) -> Capacitor_SMD:C_0402_1005Metric
- L2: renamed from L5; footprint (none) -> Inductor_SMD:L_0402_1005Metric
- L3: renamed from L6; footprint (none) -> Inductor_SMD:L_0402_1005Metric
Changed lines of the file:
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@@
 		(dnp no)
 		(fields_autoplaced yes)
-		(property "Reference" "C13"
+		(property "Reference" "C17"
 			(at 161.29 106.6799 0)
 			(effects
@@
 			)
 		)
-		(property "Footprint" ""
+		(property "Footprint" "Capacitor_SMD:C_0402_1005Metric"
 			(at 158.4452 111.76 0)
 			(effects
@@
 			(project "Senior Project"
 				(path "/16f8cce7-467e-4342-b55a-00af81cd6f69/b83b2aad-ec0d-4434-a2c8-9afe2bddf11d"
-					(reference "C13")
+					(reference "C17")
 					(unit 1)
 				)
@@
 		(dnp no)
 		(fields_autoplaced yes)
-		(property "Reference" "C11"
+		(property "Reference" "C15"
 			(at 140.97 96.5199 0)
 			(effects
@@
 			)
 		)
-		(property "Footprint" ""
+		(property "Footprint" "Capacitor_SMD:C_0402_1005Metric"
 			(at 138.1252 101.6 0)
 			(effects
@@
 			(project "Senior Project"
 				(path "/16f8cce7-467e-4342-b55a-00af81cd6f69/b83b2aad-ec0d-4434-a2c8-9afe2bddf11d"
-					(reference "C11")
+					(reference "C15")
 					(unit 1)
 				)
@@
 		(dnp no)
 		(fields_autoplaced yes)
-		(property "Reference" "#PWR021"
+		(property "Reference" "#PWR029"
 			(at 137.16 110.49 0)
 			(effects
@@
 			(project "Senior Project"
 				(path "/16f8cce7-467e-4342-b55a-00af81cd6f69/b83b2aad-ec0d-4434-a2c8-9afe2bddf11d"
-					(reference "#PWR021")
+					(reference "#PWR029")
 					(unit 1)
 				)
@@
 		(dnp no)
 		(fields_autoplaced yes)
-		(property "Reference" "#PWR024"
+		(property "Reference" "#PWR032"
 			(at 161.29 105.41 0)
 			(effects
@@
 			(project "Senior Project"
 				(path "/16f8cce7-467e-4342-b55a-00af81cd6f69/b83b2aad-ec0d-4434-a2c8-9afe2bddf11d"
-					(reference "#PWR024")
+					(reference "#PWR032")
 					(unit 1)
 				)
@@
 		(dnp no)
 		(fields_autoplaced yes)
-		(property "Reference" "AE2"
+		(property "Reference" "AE1"
 			(at 172.72 93.2814 90)
 			(effects
@@
 			)
 		)
-		(property "Footprint" ""
+		(property "Footprint" "RF_Antenna:Molex_47948-0001_2.4Ghz"
 			(at 168.91 93.98 0)
 			(effects
@@
 			(project "Senior Project"
 				(path "/16f8cce7-467e-4342-b55a-00af81cd6f69/b83b2aad-ec0d-4434-a2c8-9afe2bddf11d"
-					(reference "AE2")
+					(reference "AE1")
 					(unit 1)
 				)
@@
 		(dnp no)
 		(fields_autoplaced yes)
-		(property "Reference" "C12"
+		(property "Reference" "C16"
 			(at 151.13 96.5199 0)
 			(effects
@@
 			)
 		)
-		(property "Footprint" ""
+		(property "Footprint" "Capacitor_SMD:C_0402_1005Metric"
 			(at 148.2852 101.6 0)
 			(effects
@@
 			(project "Senior Project"
 				(path "/16f8cce7-467e-4342-b55a-00af81cd6f69/b83b2aad-ec0d-4434-a2c8-9afe2bddf11d"
-					(reference "C12")
+					(reference "C16")
 					(unit 1)
 				)
@@
 		(dnp no)
 		(fields_autoplaced yes)
-		(property "Reference" "#PWR022"
+		(property "Reference" "#PWR030"
 			(at 147.32 110.49 0)
 			(effects
@@
 			(project "Senior Project"
 				(path "/16f8cce7-467e-4342-b55a-00af81cd6f69/b83b2aad-ec0d-4434-a2c8-9afe2bddf11d"
-					(reference "#PWR022")
+					(reference "#PWR030")
 					(unit 1)
 				)
@@
 		(dnp no)
 		(fields_autoplaced yes)
-		(property "Reference" "#PWR023"
+		(property "Reference" "#PWR031"
 			(at 157.48 120.65 0)
 			(effects
@@
 			(project "Senior Project"
 				(path "/16f8cce7-467e-4342-b55a-00af81cd6f69/b83b2aad-ec0d-4434-a2c8-9afe2bddf11d"
-					(reference "#PWR023")
+					(reference "#PWR031")
 					(unit 1)
 				)
@@
 		(dnp no)
 		(fields_autoplaced yes)
-		(property "Reference" "L6"
+		(property "Reference" "L3"
 			(at 158.75 96.5199 0)
 			(effects
@@
 			)
 		)
-		(property "Footprint" ""
+		(property "Footprint" "Inductor_SMD:L_0402_1005Metric"
 			(at 157.48 97.79 0)
 			(effects
@@
 			(project "Senior Project"
 				(path "/16f8cce7-467e-4342-b55a-00af81cd6f69/b83b2aad-ec0d-4434-a2c8-9afe2bddf11d"
-					(reference "L6")
+					(reference "L3")
 					(unit 1)
 				)
@@
 		(dnp no)
 		(fields_autoplaced yes)
-		(property "Reference" "L5"
+		(property "Reference" "L2"
 			(at 142.24 88.9 90)
 			(effects
@@
 			)
 		)
-		(property "Footprint" ""
+		(property "Footprint" "Inductor_SMD:L_0402_1005Metric"
 			(at 142.24 93.98 0)
 			(effects
@@
 			(project "Senior Project"
 				(path "/16f8cce7-467e-4342-b55a-00af81cd6f69/b83b2aad-ec0d-4434-a2c8-9afe2bddf11d"
-					(reference "L5")
-					(unit 1)
-				)
+					(reference "L2")
+					(unit 1)
+				)
