File: KiCad/Radio.kicad_sch (KiCad schematic)
At the start: 2 parts, among them J1 CON-SMA-EDGE-S, U1 RFM95W-868S2

Commit message: very rough sketch layout
Parts:
- removed J1: CON-SMA-EDGE-S, CON-SMA-EDGE-S:RFSOLUTIONS_CON-SMA-EDGE-S, symbol CON-SMA-EDGE-S:CON-SMA-EDGE-S
- added AE2: Antenna_Shield, Connector_Coaxial:SMA_Samtec_SMA-J-P-H-ST-EM1_EdgeMount, symbol Device:Antenna_Shield
- U3: renamed from U1; footprint (none) -> RF_Module:HOPERF_RFM9XW_SMD
Connections:
- net GND: now also AE2.2 (Shield)
- net at U3.9 (ANT): now also AE2.1 (A)
- net +3.3V renamed +3V3
Changed lines of the file:
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@@
 	(wire
 		(pts
-			(xy 147.32 86.36) (xy 149.86 86.36)
+			(xy 130.81 106.68) (xy 130.81 109.22)
 		)
 		(stroke
@@
 	(wire
 		(pts
-			(xy 130.81 106.68) (xy 130.81 109.22)
+			(xy 113.03 88.9) (xy 120.65 88.9)
 		)
 		(stroke
@@
 	(wire
 		(pts
-			(xy 113.03 88.9) (xy 120.65 88.9)
+			(xy 135.89 106.68) (xy 135.89 109.22)
 		)
 		(stroke
@@
 		)
 	)
-	(wire
-		(pts
-			(xy 135.89 106.68) (xy 135.89 109.22)
-		)
-		(stroke
-			(width 0)
-			(type default)
-		)
-	)
 	(hierarchical_label "SCK"
 		(shape input)
@@
 	(symbol
 		(lib_id "power:GND")
-		(at 147.32 86.36 0)
+		(at 152.4 83.82 0)
 		(unit 1)
 		(exclude_from_sim no)
@@
 		(dnp no)
 		(fields_autoplaced yes)
-		(property "Reference" "#PWR02"
-			(at 147.32 92.71 0)
+		(property "Reference" "#PWR043"
+			(at 152.4 90.17 0)
 			(effects
 				(font
@@
 		)
 		(property "Value" "GND"
-			(at 147.32 91.44 0)
+			(at 152.4 88.9 0)
 			(effects
 				(font
@@
 		)
 		(property "Footprint" ""
-			(at 147.32 86.36 0)
+			(at 152.4 83.82 0)
 			(effects
 				(font
@@
 		)
 		(property "Datasheet" ""
-			(at 147.32 86.36 0)
+			(at 152.4 83.82 0)
 			(effects
 				(font
@@
 		)
 		(property "Description" "Power symbol creates a global label with name \"GND\" , ground"
-			(at 147.32 86.36 0)
+			(at 152.4 83.82 0)
 			(effects
 				(font
@@
 			(project ""
 				(path "/16f8cce7-467e-4342-b55a-00af81cd6f69/1c8bf498-9754-4bec-a707-8e930cfc3fe5"
-					(reference "#PWR02")
+					(reference "#PWR043")
 					(unit 1)
 				)
@@
 		(on_board yes)
 		(dnp no)
-		(property "Reference" "U1"
+		(property "Reference" "U3"
 			(at 135.5441 76.2 0)
 			(effects
@@
 			)
 		)
-		(property "Footprint" ""
+		(property "Footprint" "RF_Module:HOPERF_RFM9XW_SMD"
 			(at 49.53 49.53 0)
 			(effects
@@
 			(project ""
 				(path "/16f8cce7-467e-4342-b55a-00af81cd6f69/1c8bf498-9754-4bec-a707-8e930cfc3fe5"
-					(reference "U1")
+					(reference "U3")
 					(unit 1)
 				)
@@
 	)
 	(symbol
-		(lib_id "power:+3.3V")
+		(lib_id "power:+3V3")
 		(at 133.35 67.31 0)
 		(unit 1)
@@
 		(dnp no)
 		(fields_autoplaced yes)
-		(property "Reference" "#PWR01"
+		(property "Reference" "#PWR041"
 			(at 133.35 71.12 0)
 			(effects
@@
 			)
 		)
-		(property "Value" "+3.3V"
+		(property "Value" "+3V3"
 			(at 133.35 62.23 0)
 			(effects
@@
 			)
 		)
-		(property "Description" "Power symbol creates a global label with name \"+3.3V\""
+		(property "Description" "Power symbol creates a global label with name \"+3V3\""
 			(at 133.35 67.31 0)
 			(effects
@@
 			(project ""
 				(path "/16f8cce7-467e-4342-b55a-00af81cd6f69/1c8bf498-9754-4bec-a707-8e930cfc3fe5"
-					(reference "#PWR01")
-					(unit 1)
-				)
-			)
-			(project ""
-				(path "/760e4be0-0457-4cde-a6ec-d56d0abadbc7"
-					(reference "#PWR01")
+					(reference "#PWR041")
 					(unit 1)
 				)
@@
 		(dnp no)
 		(fields_autoplaced yes)
-		(property "Reference" "#PWR03"
+		(property "Reference" "#PWR042"
 			(at 133.35 119.38 0)
 			(effects
@@
 			(project ""
 				(path "/16f8cce7-467e-4342-b55a-00af81cd6f69/1c8bf498-9754-4bec-a707-8e930cfc3fe5"
-					(reference "#PWR03")
+					(reference "#PWR042")
 					(unit 1)
 				)
@@
 	)
 	(symbol
-		(lib_id "CON-SMA-EDGE-S:CON-SMA-EDGE-S")
-		(at 152.4 83.82 180)
+		(lib_id "Device:Antenna_Shield")
+		(at 149.86 78.74 0)
 		(unit 1)
 		(exclude_from_sim no)
@@
 		(dnp no)
 		(fields_autoplaced yes)
-		(property "Reference" "J1"
-			(at 157.48 83.5659 0)
-			(effects
-				(font
-					(size 1.27 1.27)
-				)
-				(justify right)
-			)
-		)
-		(property "Value" "CON-SMA-EDGE-S"
-			(at 157.48 86.1059 0)
-			(effects
-				(font
-					(size 1.27 1.27)
-				)
-				(justify right)
-			)
-		)
-		(property "Footprint" "CON-SMA-EDGE-S:RFSOLUTIONS_CON-SMA-EDGE-S"
-			(at 152.4 83.82 0)
-			(effects
-				(font
-					(size 1.27 1.27)
-				)
-				(justify bottom)
-				(hide yes)
-			)
-		)
-		(property "Datasheet" ""
-			(at 152.4 83.82 0)
-			(effects
-				(font
-					(size 1.27 1.27)
-				)
-				(hide yes)
-			)
-		)
-		(property "Description" ""
-			(at 152.4 83.82 0)
-			(effects
-				(font
-					(size 1.27 1.27)
-				)
-				(hide yes)
-			)
-		)
-		(property "PARTREV" "1"
-			(at 152.4 83.82 0)
-			(effects
-				(font
-					(size 1.27 1.27)
-				)
-				(justify bottom)
-				(hide yes)
-			)
-		)
-		(property "STANDARD" "Manufacturer Recommendations"
-			(at 152.4 83.82 0)
-			(effects
-				(font
-					(size 1.27 1.27)
-				)
-				(justify bottom)
-				(hide yes)
-			)
-		)
-		(property "MAXIMUM_PACKAGE_HEIGHT" "6.35mm"
-			(at 152.4 83.82 0)
-			(effects
-				(font
-					(size 1.27 1.27)
-				)
-				(justify bottom)
-				(hide yes)
-			)
-		)
-		(property "MANUFACTURER" "RF Solutions"
-			(at 152.4 83.82 0)
-			(effects
-				(font
-					(size 1.27 1.27)
-				)
-				(justify bottom)
-				(hide yes)
-			)
-		)
-		(pin "G1"
+		(property "Reference" "AE2"
+			(at 153.67 76.8349 0)
+			(effects
+				(font
+					(size 1.27 1.27)
+				)
+				(justify left)
+			)
+		)
+		(property "Value" "Antenna_Shield"
+			(at 153.67 79.3749 0)
+			(effects
+				(font
+					(size 1.27 1.27)
+				)
+				(justify left)
+			)
+		)
+		(property "Footprint" "Connector_Coaxial:SMA_Samtec_SMA-J-P-H-ST-EM1_EdgeMount"
+			(at 149.86 76.2 0)
+			(effects
+				(font
+					(size 1.27 1.27)
+				)
+				(hide yes)
+			)
+		)
+		(property "Datasheet" "~"
+			(at 149.86 76.2 0)
+			(effects
+				(font
+					(size 1.27 1.27)
+				)
+				(hide yes)
+			)
+		)
+		(property "Description" "Antenna with extra pin for shielding"
+			(at 149.86 78.74 0)
+			(effects
+				(font
+					(size 1.27 1.27)
+				)
+				(hide yes)
+			)
+		)
+		(pin "2"
 		)
 		(pin "1"
@@
 			(project ""
 				(path "/16f8cce7-467e-4342-b55a-00af81cd6f69/1c8bf498-9754-4bec-a707-8e930cfc3fe5"
-					(reference "J1")
-					(unit 1)
-				)
-			)
-			(project ""
-				(path "/760e4be0-0457-4cde-a6ec-d56d0abadbc7"
-					(reference "J1")
-					(unit 1)
-				)
+					(reference "AE2")
+					(unit 1)
+				)
