File: KiCad/ESP-32_Power_Coupler.kicad_sch (KiCad schematic)
At the start: 5 parts

Commit message: Reset all annotationss
Parts:
- renumbered C2 to C11, C5 to C12, C6 to C13, C7 to C14
Changed lines of the file:
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@@
 		(dnp no)
 		(fields_autoplaced yes)
-		(property "Reference" "#PWR012"
+		(property "Reference" "#PWR024"
 			(at 175.26 71.12 0)
 			(effects
@@
 			(project ""
 				(path "/16f8cce7-467e-4342-b55a-00af81cd6f69/fc885ce6-a9ef-46cc-bb26-b706458b9a56"
-					(reference "#PWR012")
+					(reference "#PWR024")
 					(unit 1)
 				)
@@
 		(dnp no)
 		(fields_autoplaced yes)
-		(property "Reference" "#PWR013"
+		(property "Reference" "#PWR025"
 			(at 185.42 71.12 0)
 			(effects
@@
 			(project ""
 				(path "/16f8cce7-467e-4342-b55a-00af81cd6f69/fc885ce6-a9ef-46cc-bb26-b706458b9a56"
-					(reference "#PWR013")
+					(reference "#PWR025")
 					(unit 1)
 				)
@@
 		(dnp no)
 		(fields_autoplaced yes)
-		(property "Reference" "C7"
+		(property "Reference" "C14"
 			(at 209.55 57.1499 0)
 			(effects
@@
 			(project "Senior Project"
 				(path "/16f8cce7-467e-4342-b55a-00af81cd6f69/fc885ce6-a9ef-46cc-bb26-b706458b9a56"
-					(reference "C7")
+					(reference "C14")
 					(unit 1)
 				)
@@
 		(dnp no)
 		(fields_autoplaced yes)
-		(property "Reference" "#PWR015"
+		(property "Reference" "#PWR028"
 			(at 205.74 71.12 0)
 			(effects
@@
 			(project ""
 				(path "/16f8cce7-467e-4342-b55a-00af81cd6f69/fc885ce6-a9ef-46cc-bb26-b706458b9a56"
-					(reference "#PWR015")
+					(reference "#PWR028")
 					(unit 1)
 				)
@@
 		(dnp no)
 		(fields_autoplaced yes)
-		(property "Reference" "C6"
+		(property "Reference" "C13"
 			(at 199.39 57.1499 0)
 			(effects
@@
 			(project "Senior Project"
 				(path "/16f8cce7-467e-4342-b55a-00af81cd6f69/fc885ce6-a9ef-46cc-bb26-b706458b9a56"
-					(reference "C6")
+					(reference "C13")
 					(unit 1)
 				)
@@
 		(dnp no)
 		(fields_autoplaced yes)
-		(property "Reference" "#PWR020"
+		(property "Reference" "#PWR027"
 			(at 205.74 50.8 0)
 			(effects
@@
 			(project ""
 				(path "/16f8cce7-467e-4342-b55a-00af81cd6f69/fc885ce6-a9ef-46cc-bb26-b706458b9a56"
-					(reference "#PWR020")
+					(reference "#PWR027")
 					(unit 1)
 				)
@@
 		(dnp no)
 		(fields_autoplaced yes)
-		(property "Reference" "C2"
+		(property "Reference" "C11"
 			(at 179.07 57.1499 0)
 			(effects
@@
 			(project ""
 				(path "/16f8cce7-467e-4342-b55a-00af81cd6f69/fc885ce6-a9ef-46cc-bb26-b706458b9a56"
-					(reference "C2")
+					(reference "C11")
 					(unit 1)
 				)
@@
 		(dnp no)
 		(fields_autoplaced yes)
-		(property "Reference" "#PWR014"
+		(property "Reference" "#PWR026"
 			(at 195.58 71.12 0)
 			(effects
@@
 			(project ""
 				(path "/16f8cce7-467e-4342-b55a-00af81cd6f69/fc885ce6-a9ef-46cc-bb26-b706458b9a56"
-					(reference "#PWR014")
+					(reference "#PWR026")
 					(unit 1)
 				)
@@
 		(dnp no)
 		(fields_autoplaced yes)
-		(property "Reference" "C5"
+		(property "Reference" "C12"
 			(at 189.23 57.1499 0)
 			(effects
@@
 			(project "Senior Project"
 				(path "/16f8cce7-467e-4342-b55a-00af81cd6f69/fc885ce6-a9ef-46cc-bb26-b706458b9a56"
-					(reference "C5")
-					(unit 1)
-				)
+					(reference "C12")
+					(unit 1)
+				)
